File: Kicad/shield_can_30_11_22.kicad_sch (KiCad schematic)
At the start: 22 parts, among them J1 GPIO, J2 Micro Android, J3 Power, J4 Analog, J5 Digital/PWM, J6 Digital/PWM, J7 Key1, U1 CD4051B

Commit message: Merge remote-tracking branch 'remote/main' update 'new pcb card'
Signed-off-by: MyAlpDroid <myalpdroid@gmail.com>
Connections:
- net GPIO[23]: now also J6.5 (Pin_5)
- net GPIO[25]: now also J6.6 (Pin_6)
- no-connect marks 20 -> 18
Other:
- note added: "2 (Int1)"
- note added: "3 (Int0)"
Changed lines of the file:
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@@
   (junction (at 224.79 129.54) (diameter 0) (color 0 0 0 0)
   )
-  (no_connect (at 190.5 88.9))
-  (no_connect (at 190.5 91.44))
   (no_connect (at 161.29 43.18))
   (no_connect (at 161.29 35.56))
@@
     (stroke (width 0) (type default) (color 0 0 0 0))
   )
-  (wire (pts (xy 73.66 45.72) (xy 100.33 45.72))
-    (stroke (width 0) (type default) (color 0 0 0 0))
-  )
   (wire (pts (xy 74.93 142.24) (xy 80.01 142.24))
     (stroke (width 0) (type default) (color 0 0 0 0))
@@
     (stroke (width 0) (type solid) (color 0 0 0 0))
   )
+  (wire (pts (xy 146.05 73.66) (xy 215.9 73.66))
+    (stroke (width 0) (type default) (color 0 0 0 0))
+  )
   (wire (pts (xy 82.55 26.67) (xy 82.55 21.59))
     (stroke (width 0) (type default) (color 0 0 0 0))
@@
     (stroke (width 0) (type default) (color 0 0 0 0))
   )
-  (wire (pts (xy 73.66 53.34) (xy 100.33 53.34))
+  (wire (pts (xy 73.66 53.34) (xy 146.05 53.34))
     (stroke (width 0) (type default) (color 0 0 0 0))
   )
@@
     (stroke (width 0) (type default) (color 0 0 0 0))
   )
+  (wire (pts (xy 218.44 88.9) (xy 218.44 63.5))
+    (stroke (width 0) (type default) (color 0 0 0 0))
+  )
   (wire (pts (xy 76.2 27.94) (xy 73.66 27.94))
     (stroke (width 0) (type solid) (color 0 0 0 0))
@@
     (stroke (width 0) (type default) (color 0 0 0 0))
   )
+  (wire (pts (xy 215.9 73.66) (xy 215.9 91.44))
+    (stroke (width 0) (type default) (color 0 0 0 0))
+  )
   (wire (pts (xy 76.2 17.78) (xy 76.2 27.94))
     (stroke (width 0) (type default) (color 0 0 0 0))
@@
     (stroke (width 0) (type solid) (color 0 0 0 0))
   )
+  (wire (pts (xy 190.5 88.9) (xy 218.44 88.9))
+    (stroke (width 0) (type default) (color 0 0 0 0))
+  )
   (wire (pts (xy 73.66 38.1) (xy 100.33 38.1))
     (stroke (width 0) (type solid) (color 0 0 0 0))
@@
     (stroke (width 0) (type default) (color 0 0 0 0))
   )
+  (wire (pts (xy 218.44 63.5) (xy 111.76 63.5))
+    (stroke (width 0) (type default) (color 0 0 0 0))
+  )
   (wire (pts (xy 191.77 38.1) (xy 191.77 55.88))
     (stroke (width 0) (type solid) (color 0 0 0 0))
@@
     (stroke (width 0) (type default) (color 0 0 0 0))
   )
-  (wire (pts (xy 100.33 52.07) (xy 100.33 53.34))
-    (stroke (width 0) (type default) (color 0 0 0 0))
-  )
   (wire (pts (xy 142.24 109.22) (xy 185.42 109.22))
     (stroke (width 0) (type default) (color 0 0 0 0))
@@
     (stroke (width 0) (type default) (color 0 0 0 0))
   )
+  (wire (pts (xy 73.66 45.72) (xy 111.76 45.72))
+    (stroke (width 0) (type default) (color 0 0 0 0))
+  )
   (wire (pts (xy 69.85 111.76) (xy 69.85 118.11))
     (stroke (width 0) (type default) (color 0 0 0 0))
@@
     (stroke (width 0) (type solid) (color 0 0 0 0))
   )
+  (wire (pts (xy 146.05 53.34) (xy 146.05 73.66))
+    (stroke (width 0) (type default) (color 0 0 0 0))
+  )
   (wire (pts (xy 142.24 45.72) (xy 161.29 45.72))
     (stroke (width 0) (type solid) (color 0 0 0 0))
@@
     (stroke (width 0) (type solid) (color 0 0 0 0))
   )
+  (wire (pts (xy 111.76 63.5) (xy 111.76 45.72))
+    (stroke (width 0) (type default) (color 0 0 0 0))
+  )
   (wire (pts (xy 161.29 48.26) (xy 158.75 48.26))
     (stroke (width 0) (type solid) (color 0 0 0 0))
+  )
+  (wire (pts (xy 215.9 91.44) (xy 190.5 91.44))
+    (stroke (width 0) (type default) (color 0 0 0 0))
   )
   (wire (pts (xy 22.86 24.13) (xy 22.86 55.88))
@@
     (effects (font (size 1.27 1.27)) (justify left bottom))
   )
+  (text "3 (Int0)" (at 194.31 88.9 0)
+    (effects (font (size 1.27 1.27)) (justify left bottom))
+  )
+  (text "2 (Int1)" (at 194.31 91.44 0)
+    (effects (font (size 1.27 1.27)) (justify left bottom))
+  )

Commit message: Merge remote-tracking branch 'remote/main' update 'readme in english'
Signed-off-by: MyAlpDroid <myalpdroid@gmail.com>
Parts:
- R6: value 470 -> 2,2k
Changed lines of the file:
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@@
       (effects (font (size 1.27 1.27)) (justify left) hide)
     )
-    (property "Value" "470" (id 1) (at 91.44 120.65 90)
+    (property "Value" "2,2k" (id 1) (at 91.44 120.65 90)
       (effects (font (size 1.27 1.27)) (justify left))
     )
@@
     )
     (path "/6f292879-6f90-4660-a0fc-221273d0ec04"
-      (reference "R6") (unit 1) (value "470") (footprint "Resistor_THT:R_Axial_DIN0207_L6.3mm_D2.5mm_P7.62mm_Horizontal")
+      (reference "R6") (unit 1) (value "2,2k") (footprint "Resistor_THT:R_Axial_DIN0207_L6.3mm_D2.5mm_P7.62mm_Horizontal")
     )
     (path "/18e103d6-daf6-45c1-a74e-d0e06857b8f9"
