File: Kicad/shield_can_30_11_22.kicad_pcb (KiCad board)
At the start: 2 copper layers, 65 x 65.6 mm, 28 parts, among them J1 GPIO, J2 Micro Android, J3 Power, J4 Analog, J5 Digital/PWM, J6 Digital/PWM, J7 Key1, U1 CD4051B

Commit message: Merge remote-tracking branch 'remote/main' update 'new pcb card'
Signed-off-by: MyAlpDroid <myalpdroid@gmail.com>
Connections:
- J6 pad 5: unconnected-(J6-Pad5) -> /GPIO[23]
- J6 pad 6: unconnected-(J6-Pad6) -> /GPIO[25]
Routing:
- net /GPIO[25]: track 0.00 -> 72.3 mm
- net /GPIO[23]: track 0.00 -> 67.6 mm
- net GND: track 194.5 -> 199.0 mm
Other:
- board text added: "100k"
- board text added: "10k"
- board text added: "15k"
- board text added: "20k"
- board text added: "22k"
- board text added: "33k"
- board text added: "4.7k"
- board text added: "470"
- board text added: "47k"
- board text added: "68k"
- board text added: "INT0"
- board text added: "INT1"

Commit message: Merge remote-tracking branch 'remote/main' update 'new pcb card'
Signed-off-by: MyAlpDroid <myalpdroid@gmail.com>
Parts:
- R6: value 470 -> 220
Other:
- board text added: "220"
- board text removed: "470"
Changed lines of the file:
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@@
       (effects (font (size 1 1) (thickness 0.15)))
     )
-    (fp_text value "470" (at 3.81 0.1) (layer "F.SilkS") hide
+    (fp_text value "220" (at 3.81 0.1) (layer "F.SilkS") hide
       (effects (font (size 1 1) (thickness 0.15)))
     )
@@
     (effects (font (size 1 1) (thickness 0.15)))
   )
-  (gr_text "470" (at 109.4 96) (layer "F.SilkS")
-    (effects (font (size 1 1) (thickness 0.15)))
-  )
+  (gr_text "220" (at 109.4 96) (layer "F.SilkS")
+    (effects (font (size 1 1) (thickness 0.15)))
+  )

Commit message: Merge remote-tracking branch 'remote/main' update 'readme in english'
Signed-off-by: MyAlpDroid <myalpdroid@gmail.com>
Parts:
- R6: value 220 -> 2,2K
Other:
- board text added: "2,2k"
- board text removed: "220"
Changed lines of the file:
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@@
       (effects (font (size 1 1) (thickness 0.15)))
     )
-    (fp_text value "220" (at 3.81 0.1) (layer "F.SilkS") hide
+    (fp_text value "2,2K" (at 3.81 0.1) (layer "F.SilkS") hide
       (effects (font (size 1 1) (thickness 0.15)))
     )
@@
     (effects (font (size 1 1) (thickness 0.15)))
   )
-  (gr_text "220" (at 109.4 96) (layer "F.SilkS")
-    (effects (font (size 1 1) (thickness 0.15)))
-  )
+  (gr_text "2,2k" (at 109.4 96) (layer "F.SilkS")
+    (effects (font (size 1 1) (thickness 0.15)))
+  )

Commit message: Merge remote-tracking branch 'remote/main' update 'radio and internet source to cluster'
Signed-off-by: MyAlpDroid <myalpdroid@gmail.com>
Parts:
- J3, J6: footprint Connector_PinSocket_2.54mm:PinSocket_1x08_P2.54mm_Vertical -> Connector_PinHeader_2.54mm:PinHeader_1x08_P2.54mm_Vertical
- J4: footprint Connector_PinSocket_2.54mm:PinSocket_1x06_P2.54mm_Vertical -> Connector_PinHeader_2.54mm:PinHeader_1x06_P2.54mm_Vertical
- J5: footprint Connector_PinSocket_2.54mm:PinSocket_1x10_P2.54mm_Vertical -> Connector_PinHeader_2.54mm:PinHeader_1x10_P2.54mm_Vertical
Connections:
- J3 pad 2: /IOREF -> (no net)
- J3 pad 3: unconnected-(J3-Pad3) -> (no net)
- J3 pad 4: unconnected-(J3-Pad4) -> (no net)
- J3 pad 5: +5V -> (no net)
- J3 pad 6: GND -> (no net)
- J3 pad 7: GND -> (no net)
- J3 pad 8: /Vin -> (no net)
