File: Kicad/_autosave-shield_can_30_11_22.kicad_pcb (KiCad board)
At the start: 2 copper layers, 65 x 65.6 mm, 28 parts, among them J1 GPIO, J2 Micro Android, J3 Power, J4 Analog, J5 Digital/PWM, J6 Digital/PWM, J7 Key1, U1 CD4051B

Commit message: Merge remote-tracking branch 'remote/main' update 'readme in english'
Signed-off-by: MyAlpDroid <myalpdroid@gmail.com>
Parts:
- J1: footprint Connector_PinSocket_2.54mm:PinSocket_2x20_P2.54mm_Vertical -> Connector_PinHeader_2.54mm:PinHeader_2x20_P2.54mm_Vertical
- moved J1 3.05 mm to (147.0, 55.5)
